File: ES-PUNKU2-0100/ES-PUNKU2-0100.kicad_pcb (KiCad board)
At the start: 2 copper layers, 87 x 66 mm, 80 parts, among them J1 PROGRAMACION, J10 SERIAL, J11 ALARMA, J2 12VDC, J3 BOOT, J4 Micro_SD_Card, J5 PULSADOR, J6 SENSOR, J7 CERRADURA, J8 RFID, J9 CONF, K1 RELE, Q1 BC817, Q2 IRF7309IPBF, Q3 IRF7309IPBF, Q4 BC817, Q5 2N7002P, Q6 2N7002P, Q7 2N7002P, U1 LM2575S5, U2 ESP32-WROOM-32D, U3 LD1117S33, U4 MCP7940N, U5 LTV-816S, U6 LTV-816S, Y1 32,768KHz

Commit message: Correcciones finales
Parts:
- moved C1 0.75 mm to (67.0, 83.0)
- moved D2 0.62 mm to (67.0, 72.8)
Routing:
- net GND: track 738.2 -> 581.9 mm, vias 9 -> 15
- net /Perifericos/ALARMA: track 39.4 -> 47.7 mm
- net /Perifericos/PULSADOR: track 70.8 -> 64.5 mm
- net /Perifericos/SENSOR: track 77.1 -> 71.5 mm
- net /Procesador/I2C_SDA: track 60.7 -> 55.1 mm
- net +3V3: track 270.2 -> 265.3 mm
- net +12V: track 214.1 -> 209.3 mm
- net /Procesador/I2C_SCL: track 53.2 -> 48.6 mm
- net /Procesador/SD_CLK: track 44.6 -> 40.0 mm
- net /Perifericos/RFID_MISO: track 29.0 -> 25.4 mm
- net /Procesador/SD_MOSI: track 37.8 -> 34.9 mm
- net /Perifericos/INVERSA: track 75.8 -> 73.1 mm
- net /Perifericos/DIRECTA: track 82.7 -> 80.3 mm
- net /Perifericos/RFID_CLK: track 21.8 -> 19.9 mm
- net +5V: track 90.2 -> 88.9 mm
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- added copper zone on B.Cu, net GND
- added copper zone on F.Cu, net GND
